Commit message: 先端追加

File: urdf/SCARA_sample.urdf (robot description, URDF)
Before this commit: robot my_SCARA, 4 links, 3 joints
Links:
- added link hand_link, mass 0.3; collision cylinder length=0.02 radius=0.05; visual cylinder length=0.02 radius=0.05
Joints:
- added joint arm2_hand: type fixed, parent arm2_link, child hand_link, origin xyz=0.5 0 0 rpy=0 0 0

Commit message: ちょっと変更

File: urdf/SCARA_sample.urdf (robot description, URDF)
Before this commit: robot my_SCARA, 5 links, 4 joints
Joints:
- joint arm2_hand: origin xyz=0.5 0 0 rpy=0 0 0 -> xyz=0.5 0 -0.01 rpy=0 0 0
