Commit message: いろいろパーツ追加

File: Catch2022_sim/urdf/SCARA_sample.urdf (robot description, URDF)
Before this commit: robot my_SCARA, 5 links, 4 joints
Links:
- removed link hand_link
- added link lefthand_link; visual cylinder length=0.01 radius=0.05
- added link linear_link; visual box size=0.1 0.1 0.4
- added link righthand_link; visual cylinder length=0.01 radius=0.05
- added link wrist_link; visual box size=0.3 0.1 0.04
- link arm1_link: mass 0.6 -> None; geometry visual box size=0.1 0.7 0.1
- link arm2_link: mass 0.6 -> None; geometry visual box size=0.1 0.65 0.1
- link stand_link: mass 10 -> None; geometry visual box size=0.7 0.3 0.3
Joints:
- removed joint arm2_hand
- added joint arm2_linear: type prismatic, parent arm2_link, child linear_link, origin xyz=0 0.65 0 rpy=0 0 0, axis 0 0 1, limit lower=-0.15 upper=0.15 effort=10 velocity=10
- added joint linear_wrist: type revolute, parent linear_link, child wrist_link, origin xyz=0 0 -0.22 rpy=0 0 0, axis 0 0 1, limit lower=-1.57075 upper=1.57075 effort=10 velocity=10
- added joint wrist_left: type fixed, parent wrist_link, child lefthand_link, origin xyz=-0.1 0 -0.025 rpy=0 0 0
- added joint wrist_right: type fixed, parent wrist_link, child righthand_link, origin xyz=0.1 0 -0.025 rpy=0 0 0
- joint arm1_arm2: origin xyz=0.5 0 0.0125 rpy=0 0 0 -> xyz=0 0.6 0.1 rpy=0 0 0
- joint base_stand: origin xyz=0 0 0.1 rpy=0 0 0 -> xyz=0 0 0.15 rpy=0 0 0
- joint stand_arm1: origin xyz=0 0 0.125 rpy=0 0 0 -> xyz=0 0 0.2 rpy=0 0 0

Commit message: nya

File: Catch2022_sim/urdf/SCARA_sample.urdf (robot description, URDF)
Before this commit: robot my_SCARA, 8 links, 7 joints
Links:
- link stand_link: geometry collision box size=0.7 0.3 0.3; visual box size=0.7 0.3 0.3

Commit message: gazeboで映るようにした

File: Catch2022_sim/urdf/SCARA_sample.urdf (robot description, URDF)
Before this commit: robot my_SCARA, 8 links, 7 joints
Links:
- link arm1_link: mass None -> 1.5; geometry collision box size=0.1 0.7 0.1; visual box size=0.1 0.7 0.1
- link arm2_link: mass None -> 1.5; geometry collision box size=0.1 0.65 0.1; visual box size=0.1 0.65 0.1
- link lefthand_link: mass None -> 0.3; geometry collision cylinder length=0.01 radius=0.05; visual cylinder length=0.01 radius=0.05
- link linear_link: mass None -> 1.3; geometry collision box size=0.1 0.1 0.4; visual box size=0.1 0.1 0.4
- link righthand_link: mass None -> 0.3; geometry collision cylinder length=0.01 radius=0.05; visual cylinder length=0.01 radius=0.05
- link stand_link: mass None -> 100
- link wrist_link: mass None -> 0.1; geometry collision box size=0.3 0.1 0.04; visual box size=0.3 0.1 0.04

Commit message: nya

File: Catch2022_sim/urdf/SCARA_sample.urdf (robot description, URDF)
Before this commit: robot my_SCARA, 8 links, 7 joints
Links:
- added link camera_link; collision box size=0.094 0.071 0.043; visual box size=0.094 0.071 0.043
- link arm2_link: geometry collision box size=0.1 0.65 0.1; visual box size=0.1 0.35 0.1
Joints:
- added joint linear_camera: type fixed, parent linear_link, child camera_link, origin xyz=0 0.097  0
- joint arm2_linear: origin xyz=0 0.65 0 rpy=0 0 0 -> xyz=0 0.35 0 rpy=0 0 0

Commit message: rvizにカメラの形をした物体を取り付けました

File: Catch2022_sim/urdf/SCARA_sample.urdf (robot description, URDF)
Before this commit: robot my_SCARA, 9 links, 8 joints
Links:
- link camera_link: mass None -> 0.168
Joints:
- joint linear_camera: origin xyz=0 0.097  0 -> xyz=0 0.0715  0 rpy=1.57 0 0
