Commit message: CHANGE : アームがガタガタになるバグの修正 赤青コーナーの座標の違いに対処

File: catch2022_sim/urdf/SCARA_sample.urdf (robot description, URDF)
Before this commit: robot my_SCARA, 8 links, 7 joints
Links:
- link stand_link: geometry visual box size=0.7 0.3 0.3

Commit message: CHANGE: バグ修正

File: catch2022_sim/urdf/SCARA_sample.urdf (robot description, URDF)
Before this commit: robot my_SCARA, 8 links, 7 joints
Links:
- link wrist_link: geometry visual box size=0.3 0.1 0.04
Joints:
- joint wrist_left: origin xyz=0 -0.1 -0.025 rpy=0 0 0 -> xyz=-0.1 -0 -0.025 rpy=0 0 0
- joint wrist_right: origin xyz=0 0.1 -0.025 rpy=0 0 0 -> xyz=0.1 0 -0.025 rpy=0 0 0
